File: hardware/bypass.sch (KiCad schematic (older format))
At the start: 10 parts, among them Q1 BSS138

Commit message: Re-Annotate
Parts:
- renumbered C12 to C13, C13 to C14, R10 to R2, R12 to R3, R13 to R4, R14 to R5, R15 to R6

Commit message: Add some component fields; Change 10uF footprint
Parts:
- C13, C14: Manufacturer (none) -> Murata; Manufacturer Part Number (none) -> GRM188R71E104KA01D; Supplier (none) -> Mouser; Supplier Link (none) -> http://eu.mouser.com/ProductDetail/Murata-Electronics/GRM18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; Supplier Part Number (none) -> 81-GRM39X104K25
- D2: Manufacturer (none) -> Diodes Incorporated; Manufacturer Link (none) -> http://www.diodes.com/catalog/Switching_Diodes_5/1N4148W_28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; Manufacturer Part Number (none) -> 1N4148W-7-F; Part Number 78-1N4148W-E3-08 -> (none); Supplier Link (none) -> http://eu.mouser.com/ProductDetail/Diodes-Incorporated/1N41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; Supplier Part Number (none) -> 621-1N4148W-F
- Q1: Manufacturer (none) -> Fairchild; Manufacturer Part Number (none) -> BSS138; Part Number 512-BSS138 -> (none); Supplier Link (none) -> http://eu.mouser.com/ProductDetail/Fairchild-Semiconductor/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; Supplier Part Number (none) -> 512-BSS138
- R2, R3, R4: Manufacturer (none) -> Vishay/Dale; Manufacturer Link (none) -> http://www.vishay.com/resistors-fixed/list/product-20011/; Manufacturer Part Number (none) -> CRCW0603100MJPEAHR; Supplier (none) -> Mouser; Supplier Link (none) -> http://eu.mouser.com/ProductDetail/Vishay-Dale/CRCW0603100M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; Supplier Part Number (none) -> 71-CRCW0603100MJPEA
- R6: Manufacturer (none) -> Vishay/Dale; Manufacturer Link (none) -> http://www.vishay.com/resistors-fixed/list/product-20011/; Manufacturer Part Number (none) -> CRCW060310K0JNEA; Supplier (none) -> Mouser; Supplier Link (none) -> http://eu.mouser.com/ProductDetail/Vishay-Dale/CRCW060310K0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; Supplier Part Number (none) -> 71-CRCW0603J-10K-E3
- REL1: Link http://www.mouser.de/ProductDetail/Omron-Electronics/G6K-2P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 -> (none); Manufacturer (none) -> Omron; Manufacturer Part Number (none) -> G6K-2P-Y-DC5; Part Number 653-G6K-2P-DC5 -> (none); Supplier Link (none) -> http://eu.mouser.com/ProductDetail/Omron-Electronics/G6K-2P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; Supplier Part Number (none) -> 653-G6K-2P-Y-DC5
Changed lines of the file:
@@
 F 1 "Omron G6K-2P-5VCD" H 8050 3600 60  0000 C CNN
 F 2 "uMIDI-switcher:Omron_G6K-2P" H 8050 3300 60  0001 C CNN
-F 3 "" H 8050 3300 60  0000 C CNN
-F 4 "Mouser" H 8050 3300 60  0001 C CNN "Supplier"
-F 5 "653-G6K-2P-DC5" H 8050 3300 60  0001 C CNN "Part Number"
-F 6 "http://www.mouser.de/ProductDetail/Omron-Electronics/G6K-2P-DC5/?qs=sGAEpiMZZMs3UE%252bXNiFaVBrMwKMEuUpxYUmZBiw8UvA%3d" H 8050 3300 60  0001 C CNN "Link"
+F 3 "https://www.omron.com/ecb/products/pdf/en-g6k.pdf" H 8050 3500 60  0001 C CNN
+F 4 "Mouser" H 8050 3500 60  0001 C CNN "Supplier"
+F 5 "653-G6K-2P-Y-DC5" H 8050 3500 60  0001 C CNN "Supplier Part Number"
+F 6 "http://eu.mouser.com/ProductDetail/Omron-Electronics/G6K-2P-Y-DC5/?qs=sGAEpiMZZMs3UE%252bXNiFaVELplwtkvP6Y68aMqtMDJ8w%3d" H 8050 3500 60  0001 C CNN "Supplier Link"
+F 7 "Omron" H 8050 3500 60  0001 C CNN "Manufacturer"
+F 8 "G6K-2P-Y-DC5" H 8050 3500 60  0001 C CNN "Manufacturer Part Number"
 	1    8050 3300
 	0    1    1    0
@@
 F 1 "Omron G6K-2P-5VCD" H 3700 3500 60  0001 C CNN
 F 2 "uMIDI-switcher:Omron_G6K-2P" H 3700 3800 60  0001 C CNN
-F 3 "" H 3700 3800 60  0000 C CNN
-F 4 "Mouser" H 8050 3300 60  0001 C CNN "Supplier"
-F 5 "653-G6K-2P-DC5" H 8050 3300 60  0001 C CNN "Part Number"
-F 6 "http://www.mouser.de/ProductDetail/Omron-Electronics/G6K-2P-DC5/?qs=sGAEpiMZZMs3UE%252bXNiFaVBrMwKMEuUpxYUmZBiw8UvA%3d" H 8050 3300 60  0001 C CNN "Link"
+F 3 "https://www.omron.com/ecb/products/pdf/en-g6k.pdf" H 3700 4000 60  0001 C CNN
+F 4 "Mouser" H 3700 4000 60  0001 C CNN "Supplier"
+F 5 "653-G6K-2P-Y-DC5" H 3700 4000 60  0001 C CNN "Supplier Part Number"
+F 6 "http://eu.mouser.com/ProductDetail/Omron-Electronics/G6K-2P-Y-DC5/?qs=sGAEpiMZZMs3UE%252bXNiFaVELplwtkvP6Y68aMqtMDJ8w%3d" H 3700 4000 60  0001 C CNN "Supplier Link"
+F 7 "Omron" H 3700 4000 60  0001 C CNN "Manufacturer"
+F 8 "G6K-2P-Y-DC5" H 3700 4000 60  0001 C CNN "Manufacturer Part Number"
 	2    3700 3800
 	1    0    0    1
@@
 F 1 "Omron G6K-2P-5VCD" H 4850 4150 60  0001 C CNN
 F 2 "uMIDI-switcher:Omron_G6K-2P" H 5200 3800 60  0001 C CNN
-F 3 "" H 5200 3800 60  0000 C CNN
-F 4 "Mouser" H 8050 3300 60  0001 C CNN "Supplier"
-F 5 "653-G6K-2P-DC5" H 8050 3300 60  0001 C CNN "Part Number"
-F 6 "http://www.mouser.de/ProductDetail/Omron-Electronics/G6K-2P-DC5/?qs=sGAEpiMZZMs3UE%252bXNiFaVBrMwKMEuUpxYUmZBiw8UvA%3d" H 8050 3300 60  0001 C CNN "Link"
+F 3 "https://www.omron.com/ecb/products/pdf/en-g6k.pdf" H 5200 4000 60  0001 C CNN
+F 4 "Mouser" H 5200 4000 60  0001 C CNN "Supplier"
+F 5 "653-G6K-2P-Y-DC5" H 5200 4000 60  0001 C CNN "Supplier Part Number"
+F 6 "http://eu.mouser.com/ProductDetail/Omron-Electronics/G6K-2P-Y-DC5/?qs=sGAEpiMZZMs3UE%252bXNiFaVELplwtkvP6Y68aMqtMDJ8w%3d" H 5200 4000 60  0001 C CNN "Supplier Link"
+F 7 "Omron" H 5200 4000 60  0001 C CNN "Manufacturer"
+F 8 "G6K-2P-Y-DC5" H 5200 4000 60  0001 C CNN "Manufacturer Part Number"
 	3    5200 3800
 	-1   0    0    1
@@
 F 1 "100M" V 4200 4150 50  0000 C CNN
 F 2 "Resistors_SMD:R_0603" V 4130 4150 30  0001 C CNN
-F 3 "" H 4200 4150 30  0000 C CNN
+F 3 "http://www.vishay.com/docs/20022/dcrcwhe3.pdf" H 4100 4150 60  0001 C CNN
+F 4 "Mouser" H 4100 4150 60  0001 C CNN "Supplier"
+F 5 "71-CRCW0603100MJPEA" H 4100 4150 60  0001 C CNN "Supplier Part Number"
+F 6 "http://eu.mouser.com/ProductDetail/Vishay-Dale/CRCW0603100MJPEAHR/?qs=sGAEpiMZZMu61qfTUdNhGwALI1ohWcNj4pxTQEkdYlc%3d" H 4100 4150 60  0001 C CNN "Supplier Link"
+F 7 "Vishay/Dale" H 4100 4150 60  0001 C CNN "Manufacturer"
+F 8 "CRCW0603100MJPEAHR" H 4100 4150 60  0001 C CNN "Manufacturer Part Number"
+F 9 "http://www.vishay.com/resistors-fixed/list/product-20011/" H 4100 4150 60  0001 C CNN "Manufacturer Link"
 	1    4200 4150
 	1    0    0    -1
@@
 F 1 "1N4148" H 7750 3200 50  0000 C CNN
 F 2 "Diodes_SMD:SOD-123" H 7750 3300 60  0001 C CNN
-F 3 "" H 7750 3300 60  0000 C CNN
-F 4 "Mouser" H 7750 3300 60  0001 C CNN "Supplier"
-F 5 "78-1N4148W-E3-08" H 7750 3300 60  0001 C CNN "Part Number"
+F 3 "http://www.diodes.com/_files/datasheets/ds30086.pdf" H 7750 3400 60  0001 C CNN
+F 4 "Mouser" H 7750 3400 60  0001 C CNN "Supplier"
+F 5 "621-1N4148W-F" H 7750 3400 60  0001 C CNN "Supplier Part Number"
+F 6 "http://eu.mouser.com/ProductDetail/Diodes-Incorporated/1N4148W-7-F/?qs=sGAEpiMZZMtoHjESLttvkiKikX2YhTL0GOrSkzAUFgM%3d" H 7750 3400 60  0001 C CNN "Supplier Link"
+F 7 "Diodes Incorporated" H 7750 3400 60  0001 C CNN "Manufacturer"
+F 8 "1N4148W-7-F" H 7750 3400 60  0001 C CNN "Manufacturer Part Number"
+F 9 "http://www.diodes.com/catalog/Switching_Diodes_5/1N4148W_2800" H 7750 3400 60  0001 C CNN "Manufacturer Link"
 	1    7750 3300
 	0    1    1    0
@@
 F 1 "100n" H 6650 3150 50  0000 L CNN
 F 2 "Capacitors_SMD:C_0603" H 6638 3100 30  0001 C CNN
-F 3 "" H 6600 3250 60  0000 C CNN
+F 3 "http://psearch.en.murata.com/capacitor/product/GRM188R71E104KA01%23.pdf" H 6650 3350 60  0001 C CNN
+F 4 "Mouser" H 3650 5050 60  0001 C CNN "Supplier"
+F 5 "81-GRM39X104K25 " H 3650 5050 60  0001 C CNN "Supplier Part Number"
+F 6 "http://eu.mouser.com/ProductDetail/Murata-Electronics/GRM188R71E104KA01D/?qs=sGAEpiMZZMs0AnBnWHyRQNOmsPzkISN0CS9R%252buxD0A8%3d" H 3650 5050 60  0001 C CNN "Supplier Link"
+F 7 "Murata" H 3650 5050 60  0001 C CNN "Manufacturer"
+F 8 "GRM188R71E104KA01D" H 3650 5050 60  0001 C CNN "Manufacturer Part Number"
 	1    6600 3250
 	1    0    0    -1
@@
 F 1 "10k" V 7507 4601 50  0000 C CNN
 F 2 "Resistors_SMD:R_0603" V 7430 4600 30  0001 C CNN
-F 3 "" H 7500 4600 30  0000 C CNN
+F 3 "http://www.vishay.com/docs/20022/dcrcwhe3.pdf" H 7580 4600 60  0001 C CNN
+F 4 "Mouser" H 7580 4600 60  0001 C CNN "Supplier"
+F 5 "71-CRCW0603J-10K-E3" H 7580 4600 60  0001 C CNN "Supplier Part Number"
+F 6 "http://eu.mouser.com/ProductDetail/Vishay-Dale/CRCW060310K0JNEA/?qs=sGAEpiMZZMu61qfTUdNhG%2fEx4adfNLScijTXbM5aXyk%3d" H 7580 4600 60  0001 C CNN "Supplier Link"
+F 7 "Vishay/Dale" H 7580 4600 60  0001 C CNN "Manufacturer"
+F 8 "CRCW060310K0JNEA" H 7580 4600 60  0001 C CNN "Manufacturer Part Number"
+F 9 "http://www.vishay.com/resistors-fixed/list/product-20011/" H 7580 4600 60  0001 C CNN "Manufacturer Link"
 	1    7500 4600
 	1    0    0    -1
@@
 F 1 "BSS138" H 7800 4400 40  0000 R CNN
 F 2 "Housings_SOT-23_SOT-143_TSOT-6:SOT-23" H 7670 4352 29  0001 C CNN
-F 3 "" H 7800 4250 60  0000 C CNN
-F 4 "Mouser" H 7800 4250 60  0001 C CNN "Supplier"
-F 5 "512-BSS138 " H 7800 4250 60  0001 C CNN "Part Number"
+F 3 "https://www.fairchildsemi.com/datasheets/BS/BSS138.pdf" H 7800 4101 60  0001 C CNN
+F 4 "Mouser" H 3650 5050 60  0001 C CNN "Supplier"
+F 5 "512-BSS138 " H 3650 5050 60  0001 C CNN "Supplier Part Number"
+F 6 "http://eu.mouser.com/ProductDetail/Fairchild-Semiconductor/BSS138/?qs=sGAEpiMZZMshyDBzk1%2fWi1qxDdW%2fXBi2IwQV99jpxW8%3d" H 3650 5050 60  0001 C CNN "Supplier Link"
+F 7 "Fairchild" H 3650 5050 60  0001 C CNN "Manufacturer"
+F 8 "BSS138" H 3650 5050 60  0001 C CNN "Manufacturer Part Number"
 	1    7800 4250
 	1    0    0    -1
@@
 F 1 "100n" H 7350 3150 50  0000 L CNN
 F 2 "Capacitors_SMD:C_0603" H 7338 3100 30  0001 C CNN
-F 3 "" H 7300 3250 60  0000 C CNN
+F 3 "http://psearch.en.murata.com/capacitor/product/GRM188R71E104KA01%23.pdf" H 7350 3350 60  0001 C CNN
+F 4 "Mouser" H 3650 5050 60  0001 C CNN "Supplier"
+F 5 "81-GRM39X104K25 " H 3650 5050 60  0001 C CNN "Supplier Part Number"
+F 6 "http://eu.mouser.com/ProductDetail/Murata-Electronics/GRM188R71E104KA01D/?qs=sGAEpiMZZMs0AnBnWHyRQNOmsPzkISN0CS9R%252buxD0A8%3d" H 3650 5050 60  0001 C CNN "Supplier Link"
+F 7 "Murata" H 3650 5050 60  0001 C CNN "Manufacturer"
+F 8 "GRM188R71E104KA01D" H 3650 5050 60  0001 C CNN "Manufacturer Part Number"
 	1    7300 3250
 	1    0    0    -1
@@
 F 1 "100M" V 4450 4150 50  0000 C CNN
 F 2 "Resistors_SMD:R_0603" V 4380 4150 30  0001 C CNN
-F 3 "" H 4450 4150 30  0000 C CNN
+F 3 "http://www.vishay.com/docs/20022/dcrcwhe3.pdf" H 4350 4150 60  0001 C CNN
+F 4 "Mouser" H 4350 4150 60  0001 C CNN "Supplier"
+F 5 "71-CRCW0603100MJPEA" H 4350 4150 60  0001 C CNN "Supplier Part Number"
+F 6 "http://eu.mouser.com/ProductDetail/Vishay-Dale/CRCW0603100MJPEAHR/?qs=sGAEpiMZZMu61qfTUdNhGwALI1ohWcNj4pxTQEkdYlc%3d" H 4350 4150 60  0001 C CNN "Supplier Link"
+F 7 "Vishay/Dale" H 4350 4150 60  0001 C CNN "Manufacturer"
+F 8 "CRCW0603100MJPEAHR" H 4350 4150 60  0001 C CNN "Manufacturer Part Number"
+F 9 "http://www.vishay.com/resistors-fixed/list/product-20011/" H 4350 4150 60  0001 C CNN "Manufacturer Link"
 	1    4450 4150
 	1    0    0    -1
@@
 F 1 "100M" V 4700 4150 50  0000 C CNN
 F 2 "Resistors_SMD:R_0603" V 4630 4150 30  0001 C CNN
-F 3 "" H 4700 4150 30  0000 C CNN
+F 3 "http://www.vishay.com/docs/20022/dcrcwhe3.pdf" H 4600 4150 60  0001 C CNN
+F 4 "Mouser" H 4600 4150 60  0001 C CNN "Supplier"
+F 5 "71-CRCW0603100MJPEA" H 4600 4150 60  0001 C CNN "Supplier Part Number"
+F 6 "http://eu.mouser.com/ProductDetail/Vishay-Dale/CRCW0603100MJPEAHR/?qs=sGAEpiMZZMu61qfTUdNhGwALI1ohWcNj4pxTQEkdYlc%3d" H 4600 4150 60  0001 C CNN "Supplier Link"
+F 7 "Vishay/Dale" H 4600 4150 60  0001 C CNN "Manufacturer"
+F 8 "CRCW0603100MJPEAHR" H 4600 4150 60  0001 C CNN "Manufacturer Part Number"
+F 9 "http://www.vishay.com/resistors-fixed/list/product-20011/" H 4600 4150 60  0001 C CNN "Manufacturer Link"
 	1    4700 4150
 	1    0    0    -1
