File: hardware/bypass.sch (KiCad schematic (older format))
At the start: 10 parts, among them Q1 BSS138

Commit message: Determine relay resistor
Parts:
- R5: value TBD -> 180; Manufacturer (none) -> Vishay/Dale; Manufacturer Link (none) -> http://www.vishay.com/resistors-fixed/list/product-20011/; Manufacturer Part Number (none) -> CRCW0603180RJNEA; Supplier (none) -> Mouser; Supplier Link (none) -> http://www.mouser.de/ProductDetail/Vishay-Dale/CRCW0603180R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; Supplier Part Number (none) -> 71-CRCW0603J-180-E3
Changed lines of the file:
@@
 AR Path="/56223A90/54E9BE9F/54D7C711" Ref="R30"  Part="1"
 F 0 "R5" V 6850 3000 50  0000 C CNN
-F 1 "TBD" V 6957 3001 50  0000 C CNN
+F 1 "180" V 6957 3001 50  0000 C CNN
 F 2 "Resistors_SMD:R_0603" V 6880 3000 30  0001 C CNN
-F 3 "" H 6950 3000 30  0000 C CNN
+F 3 "http://www.vishay.com/docs/20022/dcrcwhe3.pdf" H 6850 3000 60  0001 C CNN
+F 4 "Mouser" H 6850 3000 60  0001 C CNN "Supplier"
+F 5 "71-CRCW0603J-180-E3 " H 6850 3000 60  0001 C CNN "Supplier Part Number"
+F 6 "http://www.mouser.de/ProductDetail/Vishay-Dale/CRCW0603180RJNEA/?qs=sGAEpiMZZMu61qfTUdNhG2DpbjADlD3GH6igdLd9ZmA%3d" H 6850 3000 60  0001 C CNN "Supplier Link"
+F 7 "Vishay/Dale" H 6850 3000 60  0001 C CNN "Manufacturer"
+F 8 "CRCW0603180RJNEA" H 6850 3000 60  0001 C CNN "Manufacturer Part Number"
+F 9 "http://www.vishay.com/resistors-fixed/list/product-20011/" H 6850 3000 60  0001 C CNN "Manufacturer Link"
 	1    6950 3000
 	0    1    1    0

Commit message: Use new ldo footprint; Adapt placement
Changed lines of the file:
@@
 $Descr A4 11693 8268
 encoding utf-8
-Sheet 2 14
+Sheet 4 14
 Title ""
 Date ""
@@
 AR Path="/56223A6E/54E9BE9F/54D79A29" Ref="REL5"  Part="1"
 AR Path="/56223A7C/54E9BE9F/54D79A29" Ref="REL6"  Part="1"
-F 0 "REL1" H 8050 3500 60  0000 C CNN
+F 0 "REL6" H 8050 3500 60  0000 C CNN
 F 1 "Omron G6K-2P-5VCD" H 8050 3600 60  0000 C CNN
 F 2 "uMIDI-switcher:Omron_G6K-2P" H 8050 3300 60  0001 C CNN
@@
 AR Path="/56223A6E/54E9BE9F/54D79A79" Ref="REL5"  Part="2"
 AR Path="/56223A7C/54E9BE9F/54D79A79" Ref="REL6"  Part="2"
-F 0 "REL1" H 3700 4000 60  0000 C CNN
+F 0 "REL6" H 3700 4000 60  0000 C CNN
 F 1 "Omron G6K-2P-5VCD" H 3700 3500 60  0001 C CNN
 F 2 "uMIDI-switcher:Omron_G6K-2P" H 3700 3800 60  0001 C CNN
@@
 AR Path="/56223A6E/54E9BE9F/54D79AAA" Ref="REL5"  Part="3"
 AR Path="/56223A7C/54E9BE9F/54D79AAA" Ref="REL6"  Part="3"
-F 0 "REL1" H 5200 4000 60  0000 C CNN
+F 0 "REL6" H 5200 4000 60  0000 C CNN
 F 1 "Omron G6K-2P-5VCD" H 4850 4150 60  0001 C CNN
 F 2 "uMIDI-switcher:Omron_G6K-2P" H 5200 3800 60  0001 C CNN
@@
 AR Path="/56223A7C/54E9BE9F/54D79DA0" Ref="R22"  Part="1"
 AR Path="/56223A90/54E9BE9F/54D79DA0" Ref="R27"  Part="1"
-F 0 "R2" V 4100 4150 50  0000 C CNN
+F 0 "R22" V 4100 4150 50  0000 C CNN
 F 1 "100M" V 4200 4150 50  0000 C CNN
 F 2 "Resistors_SMD:R_0603" V 4130 4150 30  0001 C CNN
@@
 AR Path="/56223A7C/54E9BE9F/54D7A6A7" Ref="D6"  Part="1"
 AR Path="/56223A90/54E9BE9F/54D7A6A7" Ref="D7"  Part="1"
-F 0 "D2" H 7750 3400 50  0000 C CNN
+F 0 "D6" H 7750 3400 50  0000 C CNN
 F 1 "1N4148" H 7750 3200 50  0000 C CNN
 F 2 "Diodes_SMD:SOD-123" H 7750 3300 60  0001 C CNN
@@
 AR Path="/56223A7C/54E9BE9F/54D7A960" Ref="#PWR062"  Part="1"
 AR Path="/56223A90/54E9BE9F/54D7A960" Ref="#PWR069"  Part="1"
-F 0 "#PWR034" H 7900 4550 60  0001 C CNN
+F 0 "#PWR062" H 7900 4550 60  0001 C CNN
 F 1 "GND" H 7900 4650 60  0000 C CNN
 F 2 "" H 7900 4800 60  0000 C CNN
@@
 AR Path="/56223A7C/54E9BE9F/54D7AAB4" Ref="C21"  Part="1"
 AR Path="/56223A90/54E9BE9F/54D7AAB4" Ref="C23"  Part="1"
-F 0 "C13" H 6650 3350 50  0000 L CNN
+F 0 "C21" H 6650 3350 50  0000 L CNN
 F 1 "100n" H 6650 3150 50  0000 L CNN
 F 2 "Capacitors_SMD:C_0603" H 6638 3100 30  0001 C CNN
@@
 AR Path="/56223A7C/54E9BE9F/54D7AB88" Ref="#PWR063"  Part="1"
 AR Path="/56223A90/54E9BE9F/54D7AB88" Ref="#PWR070"  Part="1"
-F 0 "#PWR035" H 6600 3200 60  0001 C CNN
+F 0 "#PWR063" H 6600 3200 60  0001 C CNN
 F 1 "GND" H 6600 3300 60  0000 C CNN
 F 2 "" H 6600 3450 60  0000 C CNN
@@
 AR Path="/56223A7C/54E9BE9F/54D7ADF3" Ref="R26"  Part="1"
 AR Path="/56223A90/54E9BE9F/54D7ADF3" Ref="R31"  Part="1"
-F 0 "R6" V 7580 4600 50  0000 C CNN
+F 0 "R26" V 7580 4600 50  0000 C CNN
 F 1 "10k" V 7507 4601 50  0000 C CNN
 F 2 "Resistors_SMD:R_0603" V 7430 4600 30  0001 C CNN
@@
 AR Path="/56223A7C/54E9BE9F/54D7AECB" Ref="Q5"  Part="1"
 AR Path="/56223A90/54E9BE9F/54D7AECB" Ref="Q6"  Part="1"
-F 0 "Q1" H 7800 4101 40  0000 R CNN
+F 0 "Q5" H 7800 4101 40  0000 R CNN
 F 1 "BSS138" H 7800 4400 40  0000 R CNN
 F 2 "Housings_SOT-23_SOT-143_TSOT-6:SOT-23" H 7670 4352 29  0001 C CNN
@@
 AR Path="/56223A7C/54E9BE9F/54D7B0C5" Ref="#PWR064"  Part="1"
 AR Path="/56223A90/54E9BE9F/54D7B0C5" Ref="#PWR071"  Part="1"
-F 0 "#PWR036" H 7500 4550 60  0001 C CNN
+F 0 "#PWR064" H 7500 4550 60  0001 C CNN
 F 1 "GND" H 7500 4650 60  0000 C CNN
 F 2 "" H 7500 4800 60  0000 C CNN
@@
 AR Path="/56223A7C/54E9BE9F/54D7C711" Ref="R25"  Part="1"
 AR Path="/56223A90/54E9BE9F/54D7C711" Ref="R30"  Part="1"
-F 0 "R5" V 6850 3000 50  0000 C CNN
+F 0 "R25" V 6850 3000 50  0000 C CNN
 F 1 "180" V 6957 3001 50  0000 C CNN
 F 2 "Resistors_SMD:R_0603" V 6880 3000 30  0001 C CNN
@@
 AR Path="/56223A7C/54E9BE9F/54D7C874" Ref="C22"  Part="1"
 AR Path="/56223A90/54E9BE9F/54D7C874" Ref="C24"  Part="1"
-F 0 "C14" H 7350 3350 50  0000 L CNN
+F 0 "C22" H 7350 3350 50  0000 L CNN
 F 1 "100n" H 7350 3150 50  0000 L CNN
 F 2 "Capacitors_SMD:C_0603" H 7338 3100 30  0001 C CNN
@@
 AR Path="/56223A7C/54E9BE9F/54D7C87A" Ref="#PWR065"  Part="1"
 AR Path="/56223A90/54E9BE9F/54D7C87A" Ref="#PWR072"  Part="1"
-F 0 "#PWR037" H 7300 3200 60  0001 C CNN
+F 0 "#PWR065" H 7300 3200 60  0001 C CNN
 F 1 "GND" H 7300 3300 60  0000 C CNN
 F 2 "" H 7300 3450 60  0000 C CNN
@@
 AR Path="/56223A7C/54E9BE9F/54EA1C00" Ref="#PWR066"  Part="1"
 AR Path="/56223A90/54E9BE9F/54EA1C00" Ref="#PWR073"  Part="1"
-F 0 "#PWR038" H 4450 4250 60  0001 C CNN
+F 0 "#PWR066" H 4450 4250 60  0001 C CNN
 F 1 "GNDA" H 4450 4350 60  0000 C CNN
 F 2 "" H 4450 4500 60  0000 C CNN
@@
 AR Path="/56223A7C/54E9BE9F/54E940D4" Ref="#PWR067"  Part="1"
 AR Path="/56223A90/54E9BE9F/54E940D4" Ref="#PWR074"  Part="1"
-F 0 "#PWR039" H 6350 2800 60  0001 C CNN
+F 0 "#PWR067" H 6350 2800 60  0001 C CNN
 F 1 "+9V" H 6350 3090 60  0000 C CNN
 F 2 "" H 6350 2950 60  0000 C CNN
@@
 AR Path="/56223A7C/54E9BE9F/55F44BB0" Ref="R23"  Part="1"
 AR Path="/56223A90/54E9BE9F/55F44BB0" Ref="R28"  Part="1"
-F 0 "R3" V 4350 4150 50  0000 C CNN
+F 0 "R23" V 4350 4150 50  0000 C CNN
 F 1 "100M" V 4450 4150 50  0000 C CNN
 F 2 "Resistors_SMD:R_0603" V 4380 4150 30  0001 C CNN
@@
 AR Path="/56223A7C/54E9BE9F/55F44BF3" Ref="R24"  Part="1"
 AR Path="/56223A90/54E9BE9F/55F44BF3" Ref="R29"  Part="1"
-F 0 "R4" V 4600 4150 50  0000 C CNN
+F 0 "R24" V 4600 4150 50  0000 C CNN
 F 1 "100M" V 4700 4150 50  0000 C CNN
 F 2 "Resistors_SMD:R_0603" V 4630 4150 30  0001 C CNN

Commit message: Add 10uF caps to 9V outputs; Place and route
Changed lines of the file:
@@
 AR Path="/56223A6E/54E9BE9F/54D79A29" Ref="REL5"  Part="1"
 AR Path="/56223A7C/54E9BE9F/54D79A29" Ref="REL6"  Part="1"
-F 0 "REL6" H 8050 3500 60  0000 C CNN
+F 0 "REL2" H 8050 3500 60  0000 C CNN
 F 1 "Omron G6K-2P-5VCD" H 8050 3600 60  0000 C CNN
 F 2 "uMIDI-switcher:Omron_G6K-2P" H 8050 3300 60  0001 C CNN
@@
 AR Path="/56223A6E/54E9BE9F/54D79A79" Ref="REL5"  Part="2"
 AR Path="/56223A7C/54E9BE9F/54D79A79" Ref="REL6"  Part="2"
-F 0 "REL6" H 3700 4000 60  0000 C CNN
+F 0 "REL2" H 3700 4000 60  0000 C CNN
 F 1 "Omron G6K-2P-5VCD" H 3700 3500 60  0001 C CNN
 F 2 "uMIDI-switcher:Omron_G6K-2P" H 3700 3800 60  0001 C CNN
@@
 AR Path="/56223A6E/54E9BE9F/54D79AAA" Ref="REL5"  Part="3"
 AR Path="/56223A7C/54E9BE9F/54D79AAA" Ref="REL6"  Part="3"
-F 0 "REL6" H 5200 4000 60  0000 C CNN
+F 0 "REL2" H 5200 4000 60  0000 C CNN
 F 1 "Omron G6K-2P-5VCD" H 4850 4150 60  0001 C CNN
 F 2 "uMIDI-switcher:Omron_G6K-2P" H 5200 3800 60  0001 C CNN
@@
 AR Path="/56223A7C/54E9BE9F/54D79DA0" Ref="R22"  Part="1"
 AR Path="/56223A90/54E9BE9F/54D79DA0" Ref="R27"  Part="1"
-F 0 "R22" V 4100 4150 50  0000 C CNN
+F 0 "R27" V 4100 4150 50  0000 C CNN
 F 1 "100M" V 4200 4150 50  0000 C CNN
 F 2 "Resistors_SMD:R_0603" V 4130 4150 30  0001 C CNN
@@
 AR Path="/56223A7C/54E9BE9F/54D7A6A7" Ref="D6"  Part="1"
 AR Path="/56223A90/54E9BE9F/54D7A6A7" Ref="D7"  Part="1"
-F 0 "D6" H 7750 3400 50  0000 C CNN
+F 0 "D7" H 7750 3400 50  0000 C CNN
 F 1 "1N4148" H 7750 3200 50  0000 C CNN
 F 2 "Diodes_SMD:SOD-123" H 7750 3300 60  0001 C CNN
@@
 Connection ~ 7900 3600
 $Comp
-L GND #PWR034
+L GND #PWR42
 U 1 1 54D7A960
 P 7900 4800
-AR Path="/56223A3E/54D7A960" Ref="#PWR034"  Part="1"
-AR Path="/56223A52/54E9BE9F/54D7A960" Ref="#PWR041"  Part="1"
-AR Path="/56223A60/54E9BE9F/54D7A960" Ref="#PWR048"  Part="1"
-AR Path="/56223A6E/54E9BE9F/54D7A960" Ref="#PWR055"  Part="1"
-AR Path="/56223A7C/54E9BE9F/54D7A960" Ref="#PWR062"  Part="1"
-AR Path="/56223A90/54E9BE9F/54D7A960" Ref="#PWR069"  Part="1"
-F 0 "#PWR062" H 7900 4550 60  0001 C CNN
+AR Path="/56223A3E/54D7A960" Ref="#PWR42"  Part="1"
+AR Path="/56223A52/54E9BE9F/54D7A960" Ref="#PWR49"  Part="1"
+AR Path="/56223A60/54E9BE9F/54D7A960" Ref="#PWR56"  Part="1"
+AR Path="/56223A6E/54E9BE9F/54D7A960" Ref="#PWR63"  Part="1"
+AR Path="/56223A7C/54E9BE9F/54D7A960" Ref="#PWR70"  Part="1"
+AR Path="/56223A90/54E9BE9F/54D7A960" Ref="#PWR77"  Part="1"
+F 0 "#PWR77" H 7900 4550 60  0001 C CNN
 F 1 "GND" H 7900 4650 60  0000 C CNN
 F 2 "" H 7900 4800 60  0000 C CNN
@@
 AR Path="/56223A7C/54E9BE9F/54D7AAB4" Ref="C21"  Part="1"
 AR Path="/56223A90/54E9BE9F/54D7AAB4" Ref="C23"  Part="1"
-F 0 "C21" H 6650 3350 50  0000 L CNN
+F 0 "C23" H 6650 3350 50  0000 L CNN
 F 1 "100n" H 6650 3150 50  0000 L CNN
 F 2 "Capacitors_SMD:C_0603" H 6638 3100 30  0001 C CNN
@@
 $EndComp
 $Comp
-L GND #PWR035
+L GND #PWR39
 U 1 1 54D7AB88
 P 6600 3450
-AR Path="/56223A3E/54D7AB88" Ref="#PWR035"  Part="1"
-AR Path="/56223A52/54E9BE9F/54D7AB88" Ref="#PWR042"  Part="1"
-AR Path="/56223A60/54E9BE9F/54D7AB88" Ref="#PWR049"  Part="1"
-AR Path="/56223A6E/54E9BE9F/54D7AB88" Ref="#PWR056"  Part="1"
-AR Path="/56223A7C/54E9BE9F/54D7AB88" Ref="#PWR063"  Part="1"
-AR Path="/56223A90/54E9BE9F/54D7AB88" Ref="#PWR070"  Part="1"
-F 0 "#PWR063" H 6600 3200 60  0001 C CNN
+AR Path="/56223A3E/54D7AB88" Ref="#PWR39"  Part="1"
+AR Path="/56223A52/54E9BE9F/54D7AB88" Ref="#PWR46"  Part="1"
+AR Path="/56223A60/54E9BE9F/54D7AB88" Ref="#PWR53"  Part="1"
+AR Path="/56223A6E/54E9BE9F/54D7AB88" Ref="#PWR60"  Part="1"
+AR Path="/56223A7C/54E9BE9F/54D7AB88" Ref="#PWR67"  Part="1"
+AR Path="/56223A90/54E9BE9F/54D7AB88" Ref="#PWR74"  Part="1"
+F 0 "#PWR74" H 6600 3200 60  0001 C CNN
 F 1 "GND" H 6600 3300 60  0000 C CNN
 F 2 "" H 6600 3450 60  0000 C CNN
@@
 AR Path="/56223A7C/54E9BE9F/54D7ADF3" Ref="R26"  Part="1"
 AR Path="/56223A90/54E9BE9F/54D7ADF3" Ref="R31"  Part="1"
-F 0 "R26" V 7580 4600 50  0000 C CNN
+F 0 "R31" V 7580 4600 50  0000 C CNN
 F 1 "10k" V 7507 4601 50  0000 C CNN
 F 2 "Resistors_SMD:R_0603" V 7430 4600 30  0001 C CNN
@@
 AR Path="/56223A7C/54E9BE9F/54D7AECB" Ref="Q5"  Part="1"
 AR Path="/56223A90/54E9BE9F/54D7AECB" Ref="Q6"  Part="1"
-F 0 "Q5" H 7800 4101 40  0000 R CNN
+F 0 "Q6" H 7800 4101 40  0000 R CNN
 F 1 "BSS138" H 7800 4400 40  0000 R CNN
 F 2 "Housings_SOT-23_SOT-143_TSOT-6:SOT-23" H 7670 4352 29  0001 C CNN
@@
 	7900 4450 7900 4800
 $Comp
-L GND #PWR036
+L GND #PWR41
 U 1 1 54D7B0C5
 P 7500 4800
-AR Path="/56223A3E/54D7B0C5" Ref="#PWR036"  Part="1"
-AR Path="/56223A52/54E9BE9F/54D7B0C5" Ref="#PWR043"  Part="1"
-AR Path="/56223A60/54E9BE9F/54D7B0C5" Ref="#PWR050"  Part="1"
-AR Path="/56223A6E/54E9BE9F/54D7B0C5" Ref="#PWR057"  Part="1"
-AR Path="/56223A7C/54E9BE9F/54D7B0C5" Ref="#PWR064"  Part="1"
-AR Path="/56223A90/54E9BE9F/54D7B0C5" Ref="#PWR071"  Part="1"
-F 0 "#PWR064" H 7500 4550 60  0001 C CNN
+AR Path="/56223A3E/54D7B0C5" Ref="#PWR41"  Part="1"
+AR Path="/56223A52/54E9BE9F/54D7B0C5" Ref="#PWR48"  Part="1"
+AR Path="/56223A60/54E9BE9F/54D7B0C5" Ref="#PWR55"  Part="1"
+AR Path="/56223A6E/54E9BE9F/54D7B0C5" Ref="#PWR62"  Part="1"
+AR Path="/56223A7C/54E9BE9F/54D7B0C5" Ref="#PWR69"  Part="1"
+AR Path="/56223A90/54E9BE9F/54D7B0C5" Ref="#PWR76"  Part="1"
+F 0 "#PWR76" H 7500 4550 60  0001 C CNN
 F 1 "GND" H 7500 4650 60  0000 C CNN
 F 2 "" H 7500 4800 60  0000 C CNN
@@
 AR Path="/56223A7C/54E9BE9F/54D7C711" Ref="R25"  Part="1"
 AR Path="/56223A90/54E9BE9F/54D7C711" Ref="R30"  Part="1"
-F 0 "R25" V 6850 3000 50  0000 C CNN
+F 0 "R30" V 6850 3000 50  0000 C CNN
 F 1 "180" V 6957 3001 50  0000 C CNN
 F 2 "Resistors_SMD:R_0603" V 6880 3000 30  0001 C CNN
@@
 AR Path="/56223A7C/54E9BE9F/54D7C874" Ref="C22"  Part="1"
 AR Path="/56223A90/54E9BE9F/54D7C874" Ref="C24"  Part="1"
-F 0 "C22" H 7350 3350 50  0000 L CNN
+F 0 "C24" H 7350 3350 50  0000 L CNN
 F 1 "100n" H 7350 3150 50  0000 L CNN
 F 2 "Capacitors_SMD:C_0603" H 7338 3100 30  0001 C CNN
@@
 $EndComp
 $Comp
-L GND #PWR037
+L GND #PWR40
 U 1 1 54D7C87A
 P 7300 3450
-AR Path="/56223A3E/54D7C87A" Ref="#PWR037"  Part="1"
-AR Path="/56223A52/54E9BE9F/54D7C87A" Ref="#PWR044"  Part="1"
-AR Path="/56223A60/54E9BE9F/54D7C87A" Ref="#PWR051"  Part="1"
-AR Path="/56223A6E/54E9BE9F/54D7C87A" Ref="#PWR058"  Part="1"
-AR Path="/56223A7C/54E9BE9F/54D7C87A" Ref="#PWR065"  Part="1"
-AR Path="/56223A90/54E9BE9F/54D7C87A" Ref="#PWR072"  Part="1"
-F 0 "#PWR065" H 7300 3200 60  0001 C CNN
+AR Path="/56223A3E/54D7C87A" Ref="#PWR40"  Part="1"
+AR Path="/56223A52/54E9BE9F/54D7C87A" Ref="#PWR47"  Part="1"
+AR Path="/56223A60/54E9BE9F/54D7C87A" Ref="#PWR54"  Part="1"
+AR Path="/56223A6E/54E9BE9F/54D7C87A" Ref="#PWR61"  Part="1"
+AR Path="/56223A7C/54E9BE9F/54D7C87A" Ref="#PWR68"  Part="1"
+AR Path="/56223A90/54E9BE9F/54D7C87A" Ref="#PWR75"  Part="1"
+F 0 "#PWR75" H 7300 3200 60  0001 C CNN
 F 1 "GND" H 7300 3300 60  0000 C CNN
 F 2 "" H 7300 3450 60  0000 C CNN
@@
 Connection ~ 7300 3000
 $Comp
-L GNDA #PWR038
+L GNDA #PWR37
 U 1 1 54EA1C00
 P 4450 4500
-AR Path="/56223A3E/54EA1C00" Ref="#PWR038"  Part="1"
-AR Path="/56223A52/54E9BE9F/54EA1C00" Ref="#PWR045"  Part="1"
-AR Path="/56223A60/54E9BE9F/54EA1C00" Ref="#PWR052"  Part="1"
-AR Path="/56223A6E/54E9BE9F/54EA1C00" Ref="#PWR059"  Part="1"
-AR Path="/56223A7C/54E9BE9F/54EA1C00" Ref="#PWR066"  Part="1"
-AR Path="/56223A90/54E9BE9F/54EA1C00" Ref="#PWR073"  Part="1"
-F 0 "#PWR066" H 4450 4250 60  0001 C CNN
+AR Path="/56223A3E/54EA1C00" Ref="#PWR37"  Part="1"
+AR Path="/56223A52/54E9BE9F/54EA1C00" Ref="#PWR44"  Part="1"
+AR Path="/56223A60/54E9BE9F/54EA1C00" Ref="#PWR51"  Part="1"
+AR Path="/56223A6E/54E9BE9F/54EA1C00" Ref="#PWR58"  Part="1"
+AR Path="/56223A7C/54E9BE9F/54EA1C00" Ref="#PWR65"  Part="1"
+AR Path="/56223A90/54E9BE9F/54EA1C00" Ref="#PWR72"  Part="1"
+F 0 "#PWR72" H 4450 4250 60  0001 C CNN
 F 1 "GNDA" H 4450 4350 60  0000 C CNN
 F 2 "" H 4450 4500 60  0000 C CNN
@@
 $EndComp
 $Comp
-L +9V #PWR039
+L +9V #PWR38
 U 1 1 54E940D4
 P 6350 2950
-AR Path="/56223A3E/54E940D4" Ref="#PWR039"  Part="1"
-AR Path="/56223A52/54E9BE9F/54E940D4" Ref="#PWR046"  Part="1"
-AR Path="/56223A60/54E9BE9F/54E940D4" Ref="#PWR053"  Part="1"
-AR Path="/56223A6E/54E9BE9F/54E940D4" Ref="#PWR060"  Part="1"
-AR Path="/56223A7C/54E9BE9F/54E940D4" Ref="#PWR067"  Part="1"
-AR Path="/56223A90/54E9BE9F/54E940D4" Ref="#PWR074"  Part="1"
-F 0 "#PWR067" H 6350 2800 60  0001 C CNN
+AR Path="/56223A3E/54E940D4" Ref="#PWR38"  Part="1"
+AR Path="/56223A52/54E9BE9F/54E940D4" Ref="#PWR45"  Part="1"
+AR Path="/56223A60/54E9BE9F/54E940D4" Ref="#PWR52"  Part="1"
+AR Path="/56223A6E/54E9BE9F/54E940D4" Ref="#PWR59"  Part="1"
+AR Path="/56223A7C/54E9BE9F/54E940D4" Ref="#PWR66"  Part="1"
+AR Path="/56223A90/54E9BE9F/54E940D4" Ref="#PWR73"  Part="1"
+F 0 "#PWR73" H 6350 2800 60  0001 C CNN
 F 1 "+9V" H 6350 3090 60  0000 C CNN
 F 2 "" H 6350 2950 60  0000 C CNN
@@
 AR Path="/56223A7C/54E9BE9F/55F44BB0" Ref="R23"  Part="1"
 AR Path="/56223A90/54E9BE9F/55F44BB0" Ref="R28"  Part="1"
-F 0 "R23" V 4350 4150 50  0000 C CNN
+F 0 "R28" V 4350 4150 50  0000 C CNN
 F 1 "100M" V 4450 4150 50  0000 C CNN
 F 2 "Resistors_SMD:R_0603" V 4380 4150 30  0001 C CNN
@@
 AR Path="/56223A7C/54E9BE9F/55F44BF3" Ref="R24"  Part="1"
 AR Path="/56223A90/54E9BE9F/55F44BF3" Ref="R29"  Part="1"
-F 0 "R24" V 4600 4150 50  0000 C CNN
+F 0 "R29" V 4600 4150 50  0000 C CNN
 F 1 "100M" V 4700 4150 50  0000 C CNN
 F 2 "Resistors_SMD:R_0603" V 4630 4150 30  0001 C CNN
