File: hardware/looper.sch (KiCad schematic (older format))
At the start: 1 part, among them X7 Jack_Stacked

Commit message: Re-Annotate
Parts:
- renumbered X7 to X9
Changed lines of the file:
@@
 $EndSheet
 $Comp
-L Jack_Stacked X7
+L Jack_Stacked X9
 U 1 1 54E9CF0E
 P 6750 3250
-AR Path="/54D120FF/54E9F8A8/54E9CF0E" Ref="X7"  Part="1"
-AR Path="/54D120FF/54E9FD8E/54E9CF0E" Ref="X8"  Part="1"
-AR Path="/54D120FF/54EA08BF/54E9CF0E" Ref="X9"  Part="1"
-AR Path="/54D120FF/54EA08C5/54E9CF0E" Ref="X10"  Part="1"
-AR Path="/54D120FF/54E9BE87/54E9CF0E" Ref="X11"  Part="1"
-AR Path="/56223A90/54E9CF0E" Ref="X9"  Part="1"
 AR Path="/56223A52/54E9CF0E" Ref="X9"  Part="1"
-AR Path="/56223A60/54E9CF0E" Ref="X9"  Part="1"
-AR Path="/56223A6E/54E9CF0E" Ref="X9"  Part="1"
-AR Path="/56223A7C/54E9CF0E" Ref="X9"  Part="1"
-F 0 "X9" H 5900 5250 60  0000 C CNN
+AR Path="/56223A60/54E9CF0E" Ref="X10"  Part="1"
+AR Path="/56223A6E/54E9CF0E" Ref="X11"  Part="1"
+AR Path="/56223A7C/54E9CF0E" Ref="X12"  Part="1"
+AR Path="/56223A90/54E9CF0E" Ref="X13"  Part="1"
+F 0 "X13" H 5900 5250 60  0000 C CNN
 F 1 "Jack_Stacked" H 5850 3500 60  0000 C CNN
 F 2 "uMIDI-switcher:NSJ12HF-1" H 6750 3250 60  0001 C CNN
@@
 	4500 3700 5300 3700
 $Comp
-L GNDA #PWR038
+L GNDA #PWR40
 U 1 1 54EA1A07
 P 5100 3300
-AR Path="/54D120FF/54E9F8A8/54EA1A07" Ref="#PWR038"  Part="1"
-AR Path="/54D120FF/54E9FD8E/54EA1A07" Ref="#PWR045"  Part="1"
-AR Path="/54D120FF/54EA08BF/54EA1A07" Ref="#PWR052"  Part="1"
-AR Path="/54D120FF/54EA08C5/54EA1A07" Ref="#PWR059"  Part="1"
-AR Path="/54D120FF/54E9BE87/54EA1A07" Ref="#PWR066"  Part="1"
-AR Path="/56223A90/54EA1A07" Ref="#PWR68"  Part="1"
 AR Path="/56223A52/54EA1A07" Ref="#PWR40"  Part="1"
 AR Path="/56223A60/54EA1A07" Ref="#PWR47"  Part="1"
 AR Path="/56223A6E/54EA1A07" Ref="#PWR54"  Part="1"
 AR Path="/56223A7C/54EA1A07" Ref="#PWR61"  Part="1"
+AR Path="/56223A90/54EA1A07" Ref="#PWR68"  Part="1"
 F 0 "#PWR68" H 5100 3050 60  0001 C CNN
 F 1 "GNDA" H 5100 3150 60  0000 C CNN

Commit message: Add some component fields; Change 10uF footprint
Parts:
- X9: Link http://www.mouser.de/ProductDetail/Neutrik/NSJ12HF-1/?qs=%2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 -> (none); Manufacturer (none) -> Neutrik; Manufacturer Part Number (none) -> NSJ12HF-1; Part Number 568-NSJ12HF-1 -> (none); Supplier Link (none) -> http://www.mouser.de/ProductDetail/Neutrik/NSJ12HF-1/?qs=%2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; Supplier Part Number (none) -> 568-NSJ12HF-1
Changed lines of the file:
@@
 F 1 "Jack_Stacked" H 5850 3500 60  0000 C CNN
 F 2 "uMIDI-switcher:NSJ12HF-1" H 6750 3250 60  0001 C CNN
-F 3 "" H 6750 3250 60  0000 C CNN
-F 4 "Mouser" H 3150 2550 60  0001 C CNN "Supplier"
-F 5 "568-NSJ12HF-1 " H 3150 2550 60  0001 C CNN "Part Number"
-F 6 "http://www.mouser.de/ProductDetail/Neutrik/NSJ12HF-1/?qs=%2fha2pyFaduh94rO%252bidRgYpzOVRjO%2fmX%2foGmQWxGiJcnBKJApPofXWA%3d%3d" H 3150 2550 60  0001 C CNN "Link"
+F 3 "http://www.neutrik.com/zoolu-website/media/download/2927/Drawing+NSJ12HF-1" H 5900 5250 60  0001 C CNN
+F 4 "Mouser" H 5900 5250 60  0001 C CNN "Supplier"
+F 5 "568-NSJ12HF-1" H 5900 5250 60  0001 C CNN "Supplier Part Number"
+F 6 "http://www.mouser.de/ProductDetail/Neutrik/NSJ12HF-1/?qs=%2fha2pyFaduh94rO%252bidRgYpzOVRjO%2fmX%2foGmQWxGiJcnBKJApPofXWA%3d%3d" H 5900 5250 60  0001 C CNN "Supplier Link"
+F 7 "Neutrik" H 5900 5250 60  0001 C CNN "Manufacturer"
+F 8 "NSJ12HF-1" H 5900 5250 60  0001 C CNN "Manufacturer Part Number"
 	1    6750 3250
 	1    0    0    -1

Commit message: Straighten annotation and placement
Parts:
- renumbered X9 to X3
Changed lines of the file:
@@
 $Descr A4 11693 8268
 encoding utf-8
-Sheet 11 14
+Sheet 5 14
 Title ""
 Date ""
@@
 $EndSheet
 $Comp
-L Jack_Stacked X9
+L Jack_Stacked X3
 U 1 1 54E9CF0E
 P 6750 3250
-AR Path="/56223A52/54E9CF0E" Ref="X9"  Part="1"
-AR Path="/56223A60/54E9CF0E" Ref="X10"  Part="1"
-AR Path="/56223A6E/54E9CF0E" Ref="X11"  Part="1"
-AR Path="/56223A7C/54E9CF0E" Ref="X12"  Part="1"
-AR Path="/56223A90/54E9CF0E" Ref="X13"  Part="1"
-F 0 "X13" H 5900 5250 60  0000 C CNN
+AR Path="/56223A52/54E9CF0E" Ref="X3"  Part="1"
+AR Path="/56223A60/54E9CF0E" Ref="X4"  Part="1"
+AR Path="/56223A6E/54E9CF0E" Ref="X5"  Part="1"
+AR Path="/56223A7C/54E9CF0E" Ref="X6"  Part="1"
+AR Path="/56223A90/54E9CF0E" Ref="X2"  Part="1"
+F 0 "X4" H 5900 5250 60  0000 C CNN
 F 1 "Jack_Stacked" H 5850 3500 60  0000 C CNN
 F 2 "uMIDI-switcher:NSJ12HF-1" H 6750 3250 60  0001 C CNN
@@
 AR Path="/56223A7C/54EA1A07" Ref="#PWR061"  Part="1"
 AR Path="/56223A90/54EA1A07" Ref="#PWR068"  Part="1"
-F 0 "#PWR068" H 5100 3050 60  0001 C CNN
+F 0 "#PWR047" H 5100 3050 60  0001 C CNN
 F 1 "GNDA" H 5100 3150 60  0000 C CNN
 F 2 "" H 5100 3300 60  0000 C CNN
