File: hardware/switch.sch (KiCad schematic (older format))
At the start: 7 parts, among them Q7 BSS138

Commit message: Re-Annotate
Parts:
- renumbered C24 to C25, C25 to C26, R46 to R32, R47 to R33
Changed lines of the file:
@@
 U 1 1 54E8DEE8
 P 5400 3350
-AR Path="/54D120FF/54E8DAE1/54E8DEE8" Ref="Q7"  Part="1"
-AR Path="/54D120FF/54E90580/54E8DEE8" Ref="Q8"  Part="1"
 AR Path="/56223B06/54E8DEE8" Ref="Q7"  Part="1"
-AR Path="/56223B14/54E8DEE8" Ref="Q7"  Part="1"
-F 0 "Q7" H 5400 3201 40  0000 R CNN
+AR Path="/56223B14/54E8DEE8" Ref="Q8"  Part="1"
+F 0 "Q8" H 5400 3201 40  0000 R CNN
 F 1 "BSS138" H 5400 3500 40  0000 R CNN
 F 2 "Housings_SOT-23_SOT-143_TSOT-6:SOT-23" H 5270 3452 29  0001 C CNN
@@
 $EndComp
 $Comp
-L R R47
+L R R33
 U 1 1 54E8DF2C
 P 5100 3750
-AR Path="/54D120FF/54E8DAE1/54E8DF2C" Ref="R47"  Part="1"
-AR Path="/54D120FF/54E90580/54E8DF2C" Ref="R49"  Part="1"
-AR Path="/56223B06/54E8DF2C" Ref="R47"  Part="1"
-AR Path="/56223B14/54E8DF2C" Ref="R47"  Part="1"
-F 0 "R47" V 5180 3750 50  0000 C CNN
+AR Path="/56223B06/54E8DF2C" Ref="R33"  Part="1"
+AR Path="/56223B14/54E8DF2C" Ref="R35"  Part="1"
+F 0 "R35" V 5180 3750 50  0000 C CNN
 F 1 "10k" V 5107 3751 50  0000 C CNN
 F 2 "Resistors_SMD:R_0603" V 5030 3750 30  0001 C CNN
@@
 $EndComp
 $Comp
-L GND #PWR073
+L GND #PWR78
 U 1 1 54E8DF95
 P 5100 4100
-AR Path="/54D120FF/54E8DAE1/54E8DF95" Ref="#PWR073"  Part="1"
-AR Path="/54D120FF/54E90580/54E8DF95" Ref="#PWR078"  Part="1"
 AR Path="/56223B06/54E8DF95" Ref="#PWR78"  Part="1"
 AR Path="/56223B14/54E8DF95" Ref="#PWR83"  Part="1"
@@
 $EndComp
 $Comp
-L C C24
+L C C25
 U 1 1 54E8E18C
 P 4100 2300
-AR Path="/54D120FF/54E8DAE1/54E8E18C" Ref="C24"  Part="1"
-AR Path="/54D120FF/54E90580/54E8E18C" Ref="C26"  Part="1"
-AR Path="/56223B06/54E8E18C" Ref="C24"  Part="1"
-AR Path="/56223B14/54E8E18C" Ref="C24"  Part="1"
-F 0 "C24" H 4150 2400 50  0000 L CNN
+AR Path="/56223B06/54E8E18C" Ref="C25"  Part="1"
+AR Path="/56223B14/54E8E18C" Ref="C27"  Part="1"
+F 0 "C27" H 4150 2400 50  0000 L CNN
 F 1 "100n" H 4150 2200 50  0000 L CNN
 F 2 "Capacitors_SMD:C_0603" H 4138 2150 30  0001 C CNN
@@
 $EndComp
 $Comp
-L R R46
+L R R32
 U 1 1 54E8E1C0
 P 4450 2000
-AR Path="/54D120FF/54E8DAE1/54E8E1C0" Ref="R46"  Part="1"
-AR Path="/54D120FF/54E90580/54E8E1C0" Ref="R48"  Part="1"
-AR Path="/56223B06/54E8E1C0" Ref="R46"  Part="1"
-AR Path="/56223B14/54E8E1C0" Ref="R46"  Part="1"
-F 0 "R46" V 4530 2000 50  0000 C CNN
+AR Path="/56223B06/54E8E1C0" Ref="R32"  Part="1"
+AR Path="/56223B14/54E8E1C0" Ref="R34"  Part="1"
+F 0 "R34" V 4530 2000 50  0000 C CNN
 F 1 "TBD" V 4457 2001 50  0000 C CNN
 F 2 "Resistors_SMD:R_0603" V 4380 2000 30  0001 C CNN
@@
 $EndComp
 $Comp
-L C C25
+L C C26
 U 1 1 54E8E27F
 P 4800 2300
-AR Path="/54D120FF/54E8DAE1/54E8E27F" Ref="C25"  Part="1"
-AR Path="/54D120FF/54E90580/54E8E27F" Ref="C27"  Part="1"
-AR Path="/56223B06/54E8E27F" Ref="C25"  Part="1"
-AR Path="/56223B14/54E8E27F" Ref="C25"  Part="1"
-F 0 "C25" H 4850 2400 50  0000 L CNN
+AR Path="/56223B06/54E8E27F" Ref="C26"  Part="1"
+AR Path="/56223B14/54E8E27F" Ref="C28"  Part="1"
+F 0 "C28" H 4850 2400 50  0000 L CNN
 F 1 "100n" H 4850 2200 50  0000 L CNN
 F 2 "Capacitors_SMD:C_0603" H 4838 2150 30  0001 C CNN
@@
 $EndComp
 $Comp
-L GND #PWR074
+L GND #PWR76
 U 1 1 54E8E35E
 P 4100 2550
-AR Path="/54D120FF/54E8DAE1/54E8E35E" Ref="#PWR074"  Part="1"
-AR Path="/54D120FF/54E90580/54E8E35E" Ref="#PWR079"  Part="1"
 AR Path="/56223B06/54E8E35E" Ref="#PWR76"  Part="1"
 AR Path="/56223B14/54E8E35E" Ref="#PWR81"  Part="1"
@@
 $EndComp
 $Comp
-L +9V #PWR075
+L +9V #PWR75
 U 1 1 54E8E5BD
 P 4000 1900
-AR Path="/54D120FF/54E8DAE1/54E8E5BD" Ref="#PWR075"  Part="1"
-AR Path="/54D120FF/54E90580/54E8E5BD" Ref="#PWR080"  Part="1"
 AR Path="/56223B06/54E8E5BD" Ref="#PWR75"  Part="1"
 AR Path="/56223B14/54E8E5BD" Ref="#PWR80"  Part="1"
@@
 $EndComp
 $Comp
-L GND #PWR076
+L GND #PWR79
 U 1 1 54E8E61E
 P 5500 4100
-AR Path="/54D120FF/54E8DAE1/54E8E61E" Ref="#PWR076"  Part="1"
-AR Path="/54D120FF/54E90580/54E8E61E" Ref="#PWR081"  Part="1"
 AR Path="/56223B06/54E8E61E" Ref="#PWR79"  Part="1"
 AR Path="/56223B14/54E8E61E" Ref="#PWR84"  Part="1"
@@
 U 1 1 54E8EB7A
 P 5300 2300
-AR Path="/54D120FF/54E8DAE1/54E8EB7A" Ref="D8"  Part="1"
-AR Path="/54D120FF/54E90580/54E8EB7A" Ref="D9"  Part="1"
 AR Path="/56223B06/54E8EB7A" Ref="D8"  Part="1"
-AR Path="/56223B14/54E8EB7A" Ref="D8"  Part="1"
-F 0 "D8" H 5300 2400 50  0000 C CNN
+AR Path="/56223B14/54E8EB7A" Ref="D9"  Part="1"
+F 0 "D9" H 5300 2400 50  0000 C CNN
 F 1 "1N4148" H 5300 2200 50  0000 C CNN
 F 2 "Diodes_SMD:SOD-123" H 5300 2300 60  0001 C CNN
@@
 $EndComp
 $Comp
-L GND #PWR077
+L GND #PWR77
 U 1 1 54E8ED21
 P 4800 2550
-AR Path="/54D120FF/54E8DAE1/54E8ED21" Ref="#PWR077"  Part="1"
-AR Path="/54D120FF/54E90580/54E8ED21" Ref="#PWR082"  Part="1"
 AR Path="/56223B06/54E8ED21" Ref="#PWR77"  Part="1"
 AR Path="/56223B14/54E8ED21" Ref="#PWR82"  Part="1"
@@
 $EndComp
 $Comp
-L Relais_SPST REL7
+L Relais_SPST REL?
 U 1 1 54E8CCF9
 P 5700 2300
-AR Path="/54D120FF/54E8DAE1/54E8CCF9" Ref="REL7"  Part="1"
-AR Path="/54D120FF/54E90580/54E8CCF9" Ref="REL8"  Part="1"
+AR Path="/54D120FF/54E8DAE1/54E8CCF9" Ref="REL?"  Part="1"
+AR Path="/54D120FF/54E90580/54E8CCF9" Ref="REL?"  Part="1"
 AR Path="/56223B06/54E8CCF9" Ref="REL7"  Part="1"
-AR Path="/56223B14/54E8CCF9" Ref="REL7"  Part="1"
-F 0 "REL7" H 5700 2500 60  0000 C CNN
+AR Path="/56223B14/54E8CCF9" Ref="REL8"  Part="1"
+F 0 "REL8" H 5700 2500 60  0000 C CNN
 F 1 "Meder SIL05-1A72-71L" H 5700 2600 60  0000 C CNN
 F 2 "Socket_Strips:Socket_Strip_Straight_1x04" H 5700 2300 60  0001 C CNN
@@
 $EndComp
 $Comp
-L Relais_SPST REL7
+L Relais_SPST REL?
 U 2 1 54E8CD35
 P 6350 2300
-AR Path="/54D120FF/54E8DAE1/54E8CD35" Ref="REL7"  Part="2"
-AR Path="/54D120FF/54E90580/54E8CD35" Ref="REL8"  Part="2"
+AR Path="/54D120FF/54E8DAE1/54E8CD35" Ref="REL?"  Part="2"
+AR Path="/54D120FF/54E90580/54E8CD35" Ref="REL?"  Part="2"
 AR Path="/56223B06/54E8CD35" Ref="REL7"  Part="2"
-AR Path="/56223B14/54E8CD35" Ref="REL7"  Part="2"
-F 0 "REL7" H 6350 2500 60  0000 C CNN
+AR Path="/56223B14/54E8CD35" Ref="REL8"  Part="2"
+F 0 "REL8" H 6350 2500 60  0000 C CNN
 F 1 "Meder SIL05-1A72-71L" H 6350 2000 60  0001 C CNN
 F 2 "Socket_Strips:Socket_Strip_Straight_1x04" H 6350 2300 60  0001 C CNN

Commit message: Add some component fields; Change 10uF footprint
Parts:
- C25, C26: Manufacturer (none) -> Murata; Manufacturer Part Number (none) -> GRM188R71E104KA01D; Supplier (none) -> Mouser; Supplier Link (none) -> http://eu.mouser.com/ProductDetail/Murata-Electronics/GRM18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; Supplier Part Number (none) -> 81-GRM39X104K25
- D8: Manufacturer (none) -> Diodes Incorporated; Manufacturer Link (none) -> http://www.diodes.com/catalog/Switching_Diodes_5/1N4148W_28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; Manufacturer Part Number (none) -> 1N4148W-7-F; Part Number 78-1N4148W-E3-08 -> (none); Supplier Link (none) -> http://eu.mouser.com/ProductDetail/Diodes-Incorporated/1N41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; Supplier Part Number (none) -> 621-1N4148W-F
- Q7: Manufacturer (none) -> Fairchild; Manufacturer Part Number (none) -> BSS138; Part Number 512-BSS138 -> (none); Supplier Link (none) -> http://eu.mouser.com/ProductDetail/Fairchild-Semiconductor/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; Supplier Part Number (none) -> 512-BSS138
- R33: Manufacturer (none) -> Vishay/Dale; Manufacturer Link (none) -> http://www.vishay.com/resistors-fixed/list/product-20011/; Manufacturer Part Number (none) -> CRCW060310K0JNEA; Supplier (none) -> Mouser; Supplier Link (none) -> http://eu.mouser.com/ProductDetail/Vishay-Dale/CRCW060310K0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; Supplier Part Number (none) -> 71-CRCW0603J-10K-E3
Changed lines of the file:
@@
 F 1 "BSS138" H 5400 3500 40  0000 R CNN
 F 2 "Housings_SOT-23_SOT-143_TSOT-6:SOT-23" H 5270 3452 29  0001 C CNN
-F 3 "" H 5400 3350 60  0000 C CNN
-F 4 "Mouser" H 7800 4450 60  0001 C CNN "Supplier"
-F 5 "512-BSS138 " H 7800 4450 60  0001 C CNN "Part Number"
+F 3 "https://www.fairchildsemi.com/datasheets/BS/BSS138.pdf" H 5400 3201 60  0001 C CNN
+F 4 "Mouser" H 3650 5050 60  0001 C CNN "Supplier"
+F 5 "512-BSS138 " H 3650 5050 60  0001 C CNN "Supplier Part Number"
+F 6 "http://eu.mouser.com/ProductDetail/Fairchild-Semiconductor/BSS138/?qs=sGAEpiMZZMshyDBzk1%2fWi1qxDdW%2fXBi2IwQV99jpxW8%3d" H 3650 5050 60  0001 C CNN "Supplier Link"
+F 7 "Fairchild" H 3650 5050 60  0001 C CNN "Manufacturer"
+F 8 "BSS138" H 3650 5050 60  0001 C CNN "Manufacturer Part Number"
 	1    5400 3350
 	1    0    0    -1
@@
 F 1 "10k" V 5107 3751 50  0000 C CNN
 F 2 "Resistors_SMD:R_0603" V 5030 3750 30  0001 C CNN
-F 3 "" H 5100 3750 30  0000 C CNN
+F 3 "http://www.vishay.com/docs/20022/dcrcwhe3.pdf" H 5180 3750 60  0001 C CNN
+F 4 "Mouser" H 5180 3750 60  0001 C CNN "Supplier"
+F 5 "71-CRCW0603J-10K-E3" H 5180 3750 60  0001 C CNN "Supplier Part Number"
+F 6 "http://eu.mouser.com/ProductDetail/Vishay-Dale/CRCW060310K0JNEA/?qs=sGAEpiMZZMu61qfTUdNhG%2fEx4adfNLScijTXbM5aXyk%3d" H 5180 3750 60  0001 C CNN "Supplier Link"
+F 7 "Vishay/Dale" H 5180 3750 60  0001 C CNN "Manufacturer"
+F 8 "CRCW060310K0JNEA" H 5180 3750 60  0001 C CNN "Manufacturer Part Number"
+F 9 "http://www.vishay.com/resistors-fixed/list/product-20011/" H 5180 3750 60  0001 C CNN "Manufacturer Link"
 	1    5100 3750
 	1    0    0    -1
@@
 F 1 "100n" H 4150 2200 50  0000 L CNN
 F 2 "Capacitors_SMD:C_0603" H 4138 2150 30  0001 C CNN
-F 3 "" H 4100 2300 60  0000 C CNN
+F 3 "http://psearch.en.murata.com/capacitor/product/GRM188R71E104KA01%23.pdf" H 4150 2400 60  0001 C CNN
+F 4 "Mouser" H 3650 5050 60  0001 C CNN "Supplier"
+F 5 "81-GRM39X104K25 " H 3650 5050 60  0001 C CNN "Supplier Part Number"
+F 6 "http://eu.mouser.com/ProductDetail/Murata-Electronics/GRM188R71E104KA01D/?qs=sGAEpiMZZMs0AnBnWHyRQNOmsPzkISN0CS9R%252buxD0A8%3d" H 3650 5050 60  0001 C CNN "Supplier Link"
+F 7 "Murata" H 3650 5050 60  0001 C CNN "Manufacturer"
+F 8 "GRM188R71E104KA01D" H 3650 5050 60  0001 C CNN "Manufacturer Part Number"
 	1    4100 2300
 	1    0    0    -1
@@
 F 1 "100n" H 4850 2200 50  0000 L CNN
 F 2 "Capacitors_SMD:C_0603" H 4838 2150 30  0001 C CNN
-F 3 "" H 4800 2300 60  0000 C CNN
+F 3 "http://psearch.en.murata.com/capacitor/product/GRM188R71E104KA01%23.pdf" H 4850 2400 60  0001 C CNN
+F 4 "Mouser" H 3650 5050 60  0001 C CNN "Supplier"
+F 5 "81-GRM39X104K25 " H 3650 5050 60  0001 C CNN "Supplier Part Number"
+F 6 "http://eu.mouser.com/ProductDetail/Murata-Electronics/GRM188R71E104KA01D/?qs=sGAEpiMZZMs0AnBnWHyRQNOmsPzkISN0CS9R%252buxD0A8%3d" H 3650 5050 60  0001 C CNN "Supplier Link"
+F 7 "Murata" H 3650 5050 60  0001 C CNN "Manufacturer"
+F 8 "GRM188R71E104KA01D" H 3650 5050 60  0001 C CNN "Manufacturer Part Number"
 	1    4800 2300
 	1    0    0    -1
@@
 F 1 "1N4148" H 5300 2200 50  0000 C CNN
 F 2 "Diodes_SMD:SOD-123" H 5300 2300 60  0001 C CNN
-F 3 "" H 5300 2300 60  0000 C CNN
-F 4 "Mouser" H 5300 2300 60  0001 C CNN "Supplier"
-F 5 "78-1N4148W-E3-08 " H 5300 2300 60  0001 C CNN "Part Number"
+F 3 "http://www.diodes.com/_files/datasheets/ds30086.pdf" H 5300 2400 60  0001 C CNN
+F 4 "Mouser" H 5300 2400 60  0001 C CNN "Supplier"
+F 5 "621-1N4148W-F" H 5300 2400 60  0001 C CNN "Supplier Part Number"
+F 6 "http://eu.mouser.com/ProductDetail/Diodes-Incorporated/1N4148W-7-F/?qs=sGAEpiMZZMtoHjESLttvkiKikX2YhTL0GOrSkzAUFgM%3d" H 5300 2400 60  0001 C CNN "Supplier Link"
+F 7 "Diodes Incorporated" H 5300 2400 60  0001 C CNN "Manufacturer"
+F 8 "1N4148W-7-F" H 5300 2400 60  0001 C CNN "Manufacturer Part Number"
+F 9 "http://www.diodes.com/catalog/Switching_Diodes_5/1N4148W_2800" H 5300 2400 60  0001 C CNN "Manufacturer Link"
 	1    5300 2300
 	0    1    1    0

Commit message: Determine relay resistor
Parts:
- R32: value TBD -> 180; Manufacturer (none) -> Vishay/Dale; Manufacturer Link (none) -> http://www.vishay.com/resistors-fixed/list/product-20011/; Manufacturer Part Number (none) -> CRCW0603180RJNEA; Supplier (none) -> Mouser; Supplier Link (none) -> http://www.mouser.de/ProductDetail/Vishay-Dale/CRCW0603180R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; Supplier Part Number (none) -> 71-CRCW0603J-180-E3
Changed lines of the file:
@@
 AR Path="/56223B14/54E8E1C0" Ref="R34"  Part="1"
 F 0 "R34" V 4530 2000 50  0000 C CNN
-F 1 "TBD" V 4457 2001 50  0000 C CNN
+F 1 "180" V 4457 2001 50  0000 C CNN
 F 2 "Resistors_SMD:R_0603" V 4380 2000 30  0001 C CNN
-F 3 "" H 4450 2000 30  0000 C CNN
+F 3 "http://www.vishay.com/docs/20022/dcrcwhe3.pdf" H 4530 2000 60  0001 C CNN
+F 4 "Mouser" H 4530 2000 60  0001 C CNN "Supplier"
+F 5 "71-CRCW0603J-180-E3 " H 4530 2000 60  0001 C CNN "Supplier Part Number"
+F 6 "http://www.mouser.de/ProductDetail/Vishay-Dale/CRCW0603180RJNEA/?qs=sGAEpiMZZMu61qfTUdNhG2DpbjADlD3GH6igdLd9ZmA%3d" H 4530 2000 60  0001 C CNN "Supplier Link"
+F 7 "Vishay/Dale" H 4530 2000 60  0001 C CNN "Manufacturer"
+F 8 "CRCW0603180RJNEA" H 4530 2000 60  0001 C CNN "Manufacturer Part Number"
+F 9 "http://www.vishay.com/resistors-fixed/list/product-20011/" H 4530 2000 60  0001 C CNN "Manufacturer Link"
 	1    4450 2000
 	0    1    1    0
