File: hardware/uMIDI-switcher.sch (KiCad schematic (older format))
At the start: 29 parts, among them U1 MC7809CD, U2 MC7809CD, U3 MC7809CD, U4 MC7809CD, X1 Jack_Stacked, X10 CONN_01X02, X11 CONN_01X02, X12 CONN_01X02, X13 uMIDI GPIO, X7 Jack_Stacked, X8 12V in, X9 uMIDI Power

Commit message: Fix major footprint fuckups...
Parts:
- X10, X11, X12, X8, X9: footprint Connect:PINHEAD1-2 -> uMIDI-switcher:PINHEAD-Supply
Changed lines of the file:
@@
 $EndDescr
 $Comp
-L GND #PWR24
+L GND #PWR01
 U 1 1 54FA36B3
 P 4600 2450
-F 0 "#PWR24" H 4600 2200 60  0001 C CNN
+F 0 "#PWR01" H 4600 2200 60  0001 C CNN
 F 1 "GND" H 4600 2300 60  0000 C CNN
 F 2 "" H 4600 2450 60  0000 C CNN
@@
 NoConn ~ 4550 1500
 $Comp
-L +9V #PWR30
+L +9V #PWR02
 U 1 1 55B6A63F
 P 6550 4950
-F 0 "#PWR30" H 6550 4800 60  0001 C CNN
+F 0 "#PWR02" H 6550 4800 60  0001 C CNN
 F 1 "+9V" H 6550 5090 60  0000 C CNN
 F 2 "" H 6550 4950 60  0000 C CNN
@@
 $EndComp
 $Comp
-L +12V #PWR23
+L +12V #PWR03
 U 1 1 55B6C913
 P 4400 4950
-F 0 "#PWR23" H 4400 4800 60  0001 C CNN
+F 0 "#PWR03" H 4400 4800 60  0001 C CNN
 F 1 "+12V" H 4400 5090 60  0000 C CNN
 F 2 "" H 4400 4950 60  0000 C CNN
@@
 $EndComp
 $Comp
-L GND #PWR29
+L GND #PWR04
 U 1 1 55B70DFA
 P 6300 5500
-F 0 "#PWR29" H 6300 5250 60  0001 C CNN
+F 0 "#PWR04" H 6300 5250 60  0001 C CNN
 F 1 "GND" H 6300 5350 60  0000 C CNN
 F 2 "" H 6300 5500 60  0000 C CNN
@@
 $EndComp
 $Comp
-L GND #PWR26
+L GND #PWR05
 U 1 1 55B70E89
 P 5300 5500
-F 0 "#PWR26" H 5300 5250 60  0001 C CNN
+F 0 "#PWR05" H 5300 5250 60  0001 C CNN
 F 1 "GND" H 5300 5350 60  0000 C CNN
 F 2 "" H 5300 5500 60  0000 C CNN
@@
 $EndComp
 $Comp
-L GND #PWR27
+L GND #PWR06
 U 1 1 55B70EF4
 P 5800 5500
-F 0 "#PWR27" H 5800 5250 60  0001 C CNN
+F 0 "#PWR06" H 5800 5250 60  0001 C CNN
 F 1 "GND" H 5800 5350 60  0000 C CNN
 F 2 "" H 5800 5500 60  0000 C CNN
@@
 $EndComp
 $Comp
-L +12V #PWR1
+L +12V #PWR07
 U 1 1 55B757BE
 P 1000 5050
-F 0 "#PWR1" H 1000 4900 60  0001 C CNN
+F 0 "#PWR07" H 1000 4900 60  0001 C CNN
 F 1 "+12V" V 1000 5300 60  0000 C CNN
 F 2 "" H 1000 5050 60  0000 C CNN
@@
 $EndComp
 $Comp
-L GND #PWR11
+L GND #PWR08
 U 1 1 55B757D6
 P 2100 5500
-F 0 "#PWR11" H 2100 5250 60  0001 C CNN
+F 0 "#PWR08" H 2100 5250 60  0001 C CNN
 F 1 "GND" H 2100 5350 60  0000 C CNN
 F 2 "" H 2100 5500 60  0000 C CNN
@@
 $EndComp
 $Comp
-L GND #PWR4
+L GND #PWR09
 U 1 1 55B757DC
 P 1100 5500
-F 0 "#PWR4" H 1100 5250 60  0001 C CNN
+F 0 "#PWR09" H 1100 5250 60  0001 C CNN
 F 1 "GND" H 1100 5350 60  0000 C CNN
 F 2 "" H 1100 5500 60  0000 C CNN
@@
 $EndComp
 $Comp
-L GND #PWR8
+L GND #PWR010
 U 1 1 55B757E2
 P 1600 5500
-F 0 "#PWR8" H 1600 5250 60  0001 C CNN
+F 0 "#PWR010" H 1600 5250 60  0001 C CNN
 F 1 "GND" H 1600 5350 60  0000 C CNN
 F 2 "" H 1600 5500 60  0000 C CNN
@@
 F 0 "X10" H 2950 5250 50  0000 C CNN
 F 1 "CONN_01X02" V 3050 5100 50  0001 C CNN
-F 2 "Connect:PINHEAD1-2" H 2950 5100 60  0001 C CNN
+F 2 "uMIDI-switcher:PINHEAD-Supply" H 2950 5100 60  0001 C CNN
 F 3 "" H 2950 5100 60  0000 C CNN
 F 4 "Mouser" H 3950 5050 60  0001 C CNN "Supplier"
@@
 $EndComp
 $Comp
-L GND #PWR18
+L GND #PWR011
 U 1 1 55B757FA
 P 2700 5500
-F 0 "#PWR18" H 2700 5250 60  0001 C CNN
+F 0 "#PWR011" H 2700 5250 60  0001 C CNN
 F 1 "GND" H 2700 5350 60  0000 C CNN
 F 2 "" H 2700 5500 60  0000 C CNN
@@
 F 0 "X8" H 3350 5250 50  0000 C CNN
 F 1 "12V in" V 3450 5100 50  0001 C CNN
-F 2 "Connect:PINHEAD1-2" H 3350 5100 60  0001 C CNN
+F 2 "uMIDI-switcher:PINHEAD-Supply" H 3350 5100 60  0001 C CNN
 F 3 "" H 3350 5100 60  0000 C CNN
 F 4 "Mouser" H 4050 5050 60  0001 C CNN "Supplier"
@@
 $EndComp
 $Comp
-L GND #PWR21
+L GND #PWR012
 U 1 1 55B7738A
 P 3600 5200
-F 0 "#PWR21" H 3600 4950 60  0001 C CNN
+F 0 "#PWR012" H 3600 4950 60  0001 C CNN
 F 1 "GND" H 3600 5050 60  0000 C CNN
 F 2 "" H 3600 5200 60  0000 C CNN
@@
 $EndComp
 $Comp
-L GND #PWR22
+L GND #PWR013
 U 1 1 55B7845A
 P 4250 5500
-F 0 "#PWR22" H 4250 5250 60  0001 C CNN
+F 0 "#PWR013" H 4250 5250 60  0001 C CNN
 F 1 "GND" H 4250 5350 60  0000 C CNN
 F 2 "" H 4250 5500 60  0000 C CNN
@@
 $EndComp
 $Comp
-L +12V #PWR2
+L +12V #PWR014
 U 1 1 55F43672
 P 1000 6000
-F 0 "#PWR2" H 1000 5850 60  0001 C CNN
+F 0 "#PWR014" H 1000 5850 60  0001 C CNN
 F 1 "+12V" V 1000 6250 60  0000 C CNN
 F 2 "" H 1000 6000 60  0000 C CNN
@@
 $EndComp
 $Comp
-L GND #PWR12
+L GND #PWR015
 U 1 1 55F4368A
 P 2100 6450
-F 0 "#PWR12" H 2100 6200 60  0001 C CNN
+F 0 "#PWR015" H 2100 6200 60  0001 C CNN
 F 1 "GND" H 2100 6300 60  0000 C CNN
 F 2 "" H 2100 6450 60  0000 C CNN
@@
 $EndComp
 $Comp
-L GND #PWR5
+L GND #PWR016
 U 1 1 55F43690
 P 1100 6450
-F 0 "#PWR5" H 1100 6200 60  0001 C CNN
+F 0 "#PWR016" H 1100 6200 60  0001 C CNN
 F 1 "GND" H 1100 6300 60  0000 C CNN
 F 2 "" H 1100 6450 60  0000 C CNN
@@
 $EndComp
 $Comp
-L GND #PWR9
+L GND #PWR017
 U 1 1 55F43696
 P 1600 6450
-F 0 "#PWR9" H 1600 6200 60  0001 C CNN
+F 0 "#PWR017" H 1600 6200 60  0001 C CNN
 F 1 "GND" H 1600 6300 60  0000 C CNN
 F 2 "" H 1600 6450 60  0000 C CNN
@@
 F 0 "X11" H 2950 6200 50  0000 C CNN
 F 1 "CONN_01X02" V 3050 6050 50  0001 C CNN
-F 2 "Connect:PINHEAD1-2" H 2950 6050 60  0001 C CNN
+F 2 "uMIDI-switcher:PINHEAD-Supply" H 2950 6050 60  0001 C CNN
 F 3 "" H 2950 6050 60  0000 C CNN
 F 4 "Mouser" H 3950 5050 60  0001 C CNN "Supplier"
@@
 $EndComp
 $Comp
-L GND #PWR19
+L GND #PWR018
 U 1 1 55F436AA
 P 2700 6450
-F 0 "#PWR19" H 2700 6200 60  0001 C CNN
+F 0 "#PWR018" H 2700 6200 60  0001 C CNN
 F 1 "GND" H 2700 6300 60  0000 C CNN
 F 2 "" H 2700 6450 60  0000 C CNN
@@
 $EndComp
 $Comp
-L +12V #PWR3
+L +12V #PWR019
 U 1 1 55F4379F
 P 1000 6950
-F 0 "#PWR3" H 1000 6800 60  0001 C CNN
+F 0 "#PWR019" H 1000 6800 60  0001 C CNN
 F 1 "+12V" V 1000 7200 60  0000 C CNN
 F 2 "" H 1000 6950 60  0000 C CNN
@@
 $EndComp
 $Comp
-L GND #PWR13
+L GND #PWR020
 U 1 1 55F437B7
 P 2100 7400
-F 0 "#PWR13" H 2100 7150 60  0001 C CNN
+F 0 "#PWR020" H 2100 7150 60  0001 C CNN
 F 1 "GND" H 2100 7250 60  0000 C CNN
 F 2 "" H 2100 7400 60  0000 C CNN
@@
 $EndComp
 $Comp
-L GND #PWR6
+L GND #PWR021
 U 1 1 55F437BD
 P 1100 7400
-F 0 "#PWR6" H 1100 7150 60  0001 C CNN
+F 0 "#PWR021" H 1100 7150 60  0001 C CNN
 F 1 "GND" H 1100 7250 60  0000 C CNN
 F 2 "" H 1100 7400 60  0000 C CNN
@@
 $EndComp
 $Comp
-L GND #PWR10
+L GND #PWR022
 U 1 1 55F437C3
 P 1600 7400
-F 0 "#PWR10" H 1600 7150 60  0001 C CNN
+F 0 "#PWR022" H 1600 7150 60  0001 C CNN
 F 1 "GND" H 1600 7250 60  0000 C CNN
 F 2 "" H 1600 7400 60  0000 C CNN
@@
 F 0 "X12" H 2950 7150 50  0000 C CNN
 F 1 "CONN_01X02" V 3050 7000 50  0001 C CNN
-F 2 "Connect:PINHEAD1-2" H 2950 7000 60  0001 C CNN
+F 2 "uMIDI-switcher:PINHEAD-Supply" H 2950 7000 60  0001 C CNN
 F 3 "" H 2950 7000 60  0000 C CNN
 F 4 "Mouser" H 3950 5050 60  0001 C CNN "Supplier"
@@
 $EndComp
 $Comp
-L GND #PWR20
+L GND #PWR023
 U 1 1 55F437D7
 P 2700 7400
-F 0 "#PWR20" H 2700 7150 60  0001 C CNN
+F 0 "#PWR023" H 2700 7150 60  0001 C CNN
 F 1 "GND" H 2700 7250 60  0000 C CNN
 F 2 "" H 2700 7400 60  0000 C CNN
@@
 F 0 "X9" H 7950 5400 50  0000 C CNN
 F 1 "uMIDI Power" V 8050 5250 50  0000 C CNN
-F 2 "Connect:PINHEAD1-2" H 7950 5250 60  0001 C CNN
+F 2 "uMIDI-switcher:PINHEAD-Supply" H 7950 5250 60  0001 C CNN
 F 3 "" H 7950 5250 60  0000 C CNN
 F 4 "Mouser" H 4050 5050 60  0001 C CNN "Supplier"
@@
 $EndComp
 $Comp
-L GND #PWR33
+L GND #PWR024
 U 1 1 55FDF929
 P 7500 5500
-F 0 "#PWR33" H 7500 5250 60  0001 C CNN
+F 0 "#PWR024" H 7500 5250 60  0001 C CNN
 F 1 "GND" H 7500 5350 60  0000 C CNN
 F 2 "" H 7500 5500 60  0000 C CNN
@@
 $EndComp
 $Comp
-L GND #PWR34
+L GND #PWR025
 U 1 1 55FE932A
 P 7750 5500
-F 0 "#PWR34" H 7750 5250 60  0001 C CNN
+F 0 "#PWR025" H 7750 5250 60  0001 C CNN
 F 1 "GND" H 7750 5350 60  0000 C CNN
 F 2 "" H 7750 5500 60  0000 C CNN
@@
 Connection ~ 6650 5050
 $Comp
-L GND #PWR32
+L GND #PWR026
 U 1 1 55FED47B
 P 6650 5500
-F 0 "#PWR32" H 6650 5250 60  0001 C CNN
+F 0 "#PWR026" H 6650 5250 60  0001 C CNN
 F 1 "GND" H 6650 5350 60  0000 C CNN
 F 2 "" H 6650 5500 60  0000 C CNN
@@
 	6650 5500 6650 5450
 $Comp
-L GND #PWR25
+L GND #PWR027
 U 1 1 55FED76E
 P 4950 5500
-F 0 "#PWR25" H 4950 5250 60  0001 C CNN
+F 0 "#PWR027" H 4950 5250 60  0001 C CNN
 F 1 "GND" H 4950 5350 60  0000 C CNN
 F 2 "" H 4950 5500 60  0000 C CNN
@@
 	1150 2100 1650 2100
 $Comp
-L GNDA #PWR14
+L GNDA #PWR028
 U 1 1 56223AAC
 P 2450 3100
-F 0 "#PWR14" H 2450 2850 60  0001 C CNN
+F 0 "#PWR028" H 2450 2850 60  0001 C CNN
 F 1 "GNDA" H 2450 2950 60  0000 C CNN
 F 2 "" H 2450 3100 60  0000 C CNN
@@
 	2450 3300 2350 3300
 $Comp
-L GNDA #PWR7
+L GNDA #PWR029
 U 1 1 56223AB3
 P 1550 2700
-F 0 "#PWR7" H 1550 2450 60  0001 C CNN
+F 0 "#PWR029" H 1550 2450 60  0001 C CNN
 F 1 "GNDA" H 1550 2550 60  0000 C CNN
 F 2 "" H 1550 2700 60  0000 C CNN
@@
 $EndComp
 $Comp
-L GNDA #PWR36
+L GNDA #PWR030
 U 1 1 56223AD5
 P 9850 2700
-F 0 "#PWR36" H 9850 2450 60  0001 C CNN
+F 0 "#PWR030" H 9850 2450 60  0001 C CNN
 F 1 "GNDA" H 9850 2550 60  0000 C CNN
 F 2 "" H 9850 2700 60  0000 C CNN
@@
 	10050 1250 9750 1250
 $Comp
-L GNDA #PWR35
+L GNDA #PWR031
 U 1 1 56223AE6
 P 9850 1450
-F 0 "#PWR35" H 9850 1200 60  0001 C CNN
+F 0 "#PWR031" H 9850 1200 60  0001 C CNN
 F 1 "GNDA" H 9850 1300 60  0000 C CNN
 F 2 "" H 9850 1450 60  0000 C CNN
@@
 	4550 2300 4750 2300
 $Comp
-L GNDA #PWR31
+L GNDA #PWR032
 U 1 1 56216618
 P 6600 2050
-F 0 "#PWR31" H 6600 1800 60  0001 C CNN
+F 0 "#PWR032" H 6600 1800 60  0001 C CNN
 F 1 "GNDA" H 6600 1900 60  0000 C CNN
 F 2 "" H 6600 2050 60  0000 C CNN
@@
 $EndComp
 $Comp
-L GND #PWR28
+L GND #PWR033
 U 1 1 5621670A
 P 6300 2050
-F 0 "#PWR28" H 6300 1800 60  0001 C CNN
+F 0 "#PWR033" H 6300 1800 60  0001 C CNN
 F 1 "GND" H 6300 1900 60  0000 C CNN
 F 2 "" H 6300 2050 60  0000 C CNN
@@
 Connection ~ 2450 6000
 $Comp
-L GND #PWR16
+L GND #PWR034
 U 1 1 565749AA
 P 2450 6450
-F 0 "#PWR16" H 2450 6200 60  0001 C CNN
+F 0 "#PWR034" H 2450 6200 60  0001 C CNN
 F 1 "GND" H 2450 6300 60  0000 C CNN
 F 2 "" H 2450 6450 60  0000 C CNN
@@
 $EndComp
 $Comp
-L GND #PWR17
+L GND #PWR035
 U 1 1 56575050
 P 2450 7400
-F 0 "#PWR17" H 2450 7150 60  0001 C CNN
+F 0 "#PWR035" H 2450 7150 60  0001 C CNN
 F 1 "GND" H 2450 7250 60  0000 C CNN
 F 2 "" H 2450 7400 60  0000 C CNN
@@
 Connection ~ 2450 5050
 $Comp
-L GND #PWR15
+L GND #PWR036
 U 1 1 565760A5
 P 2450 5500
-F 0 "#PWR15" H 2450 5250 60  0001 C CNN
+F 0 "#PWR036" H 2450 5250 60  0001 C CNN
 F 1 "GND" H 2450 5350 60  0000 C CNN
 F 2 "" H 2450 5500 60  0000 C CNN
