File: hardware/uMIDI-switcher.sch (KiCad schematic (older format))
At the start: 29 parts, among them U1 MC7809CD, U2 MC7809CD, U3 MC7809CD, U4 MC7809CD, X1 Jack_Stacked, X10 CONN_01X02, X11 CONN_01X02, X12 CONN_01X02, X13 uMIDI GPIO, X7 Jack_Stacked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

Commit message: Fix faulty jack connections
Connections:
- net GNDA: now also X1.9 (TNB); no longer X1.11 (RNB), X1.4 (RB)
- no-connect marks 4 -> 7
Changed lines of the file:
@@
 	1650 1800 1550 1800
 Connection ~ 1550 1800
-Wire Wire Line
-	1650 1900 1550 1900
-Connection ~ 1550 1900
-Wire Wire Line
-	1650 2000 1550 2000
-Connection ~ 1550 2000
 $Comp
 L Jack_Stacked X7
@@
 Wire Wire Line
 	2450 5500 2450 5450
+Wire Wire Line
+	1650 2200 1550 2200
+Connection ~ 1550 2200
+NoConn ~ 1650 1900
+NoConn ~ 1650 2000
+NoConn ~ 1650 1350
 $EndSCHEMATC
